File: Hardware/Rack0/rack0/rack0.kicad_sch (KiCad schematic)
At the start: 46 parts, among them M1 Fan_4pin, M2 Fan_4pin, M4 Dosificador0, M5 Dosificador1, M6 Dosificador2, M7 Bomba_principal, Q1 BC550, Q2 BC550, Q3 BC550, U1 LM7805_TO220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

Commit message: Esquemas
Parts:
- added C9: 100nf, symbol Device:C
- added U7: HT-CT62, RF_Module:Heltec_HT-CT62, symbol RF_Module:HT-CT62
Connections:
- net GND1: now also C9.2, U7.13 (GND), U7.2 (GND), U7.21 (GND)
- net VCC_5v: now also C9.1, U7.12 (VDD)
- net UART_TX_0: now reaches STM32F103.12 (A7)
- net UART_TX_0: now also U7.9 (GPIO1)
- net UART_RX_0: now reaches STM32F103.13 (B0)
- net UART_RX_0: now also U7.8 (GPIO2)
- net UART_RX_1: now reaches STM32F114.11 (A5)
- net UART_RX_1: now also U7.6 (GPIO4)
- net UART_TX_1: now reaches STM32F114.12 (A6)
- net UART_TX_1: now also U7.5 (GPIO5)
